Commit message: add imu and gps to boy

File: falkor_quadrotor_urdf/urdf/boy.urdf.xacro (robot description, xacro)
@@ -6,4 +6,6 @@
     xmlns:xacro="http://ros.org/wiki/xacro"
 >
+  <property name="pi" value="3.1415926535897931" />
+  <include filename="$(find hector_quadrotor_controller)/urdf/quadrotor_sensors.urdf.xacro" />
   <xacro:macro name="boy_base" params="mass height width depth">
     <link name="base_link">
@@ -21,5 +23,5 @@
       </inertial>
       <visual>
-        <origin xyz="0 0 0" rpy="0 0 0" />
+        <origin xyz="0 0 0" rpy="0 0 ${pi/2}" />
         <geometry>
           <mesh filename="package://falkor_quadrotor_urdf/meshes/boy.dae"/>
@@ -36,5 +38,6 @@
       <turnGravityOff>false</turnGravityOff>
     </gazebo>
+    <quadrotor_sensors/>
   </xacro:macro>
-  <boy_base height="1.70" width="0.40" depth="0.20" mass="70" />
+  <boy_base height="1.70" width="0.80" depth="0.60" mass="70" />
 </robot>

Commit message: rename the boy's base_link to body_link so that the hector imu/gps simulated sensors don't get confused

File: falkor_quadrotor_urdf/urdf/boy.urdf.xacro (robot description, xacro)
@@ -7,7 +7,7 @@
 >
   <property name="pi" value="3.1415926535897931" />
-  <include filename="$(find hector_quadrotor_controller)/urdf/quadrotor_sensors.urdf.xacro" />
+  <include filename="$(find falkor_quadrotor_urdf)/urdf/beacon_sensors.urdf.xacro" />
   <xacro:macro name="boy_base" params="mass height width depth">
-    <link name="base_link">
+    <link name="body_link">
       <inertial>
         <mass value="${mass}" />
@@ -38,5 +38,5 @@
       <turnGravityOff>false</turnGravityOff>
     </gazebo>
-    <quadrotor_sensors/>
+    <beacon_sensors />
   </xacro:macro>
   <boy_base height="1.70" width="0.80" depth="0.60" mass="70" />

Commit message: reorganize and put the direct quad controller on js3

File: falkor_quadrotor_urdf/urdf/boy.urdf.xacro (robot description, xacro)
@@ -23,5 +23,5 @@
       </inertial>
       <visual>
-        <origin xyz="0 0 0" rpy="0 0 ${pi/2}" />
+        <origin xyz="0 0 0" rpy="0 0 -${pi/2}" />
         <geometry>
           <mesh filename="package://falkor_quadrotor_urdf/meshes/boy.dae"/>
