Commit message: rename body_link back to base_link

File: falkor_quadrotor_urdf/urdf/beacon_sensors.urdf.xacro (robot description, xacro)
@@ -11,5 +11,5 @@
         <alwaysOn>true</alwaysOn>
         <updateRate>100.0</updateRate>
-        <bodyName>body_link</bodyName>
+        <bodyName>base_link</bodyName>
         <topicName>raw_imu</topicName>
         <rpyOffsets>0 0 0</rpyOffsets> <!-- deprecated -->
@@ -25,5 +25,5 @@
         <alwaysOn>true</alwaysOn>
         <updateRate>10.0</updateRate>
-        <bodyName>body_link</bodyName>
+        <bodyName>base_link</bodyName>
         <topicName>pressure_height</topicName>
         <altimeterTopicName>altimeter</altimeterTopicName>
@@ -35,5 +35,5 @@
         <alwaysOn>true</alwaysOn>
         <updateRate>10.0</updateRate>
-        <bodyName>body_link</bodyName>
+        <bodyName>base_link</bodyName>
         <topicName>magnetic</topicName>
         <offset>0 0 0</offset>
@@ -44,5 +44,5 @@
         <alwaysOn>true</alwaysOn>
         <updateRate>4.0</updateRate>
-        <bodyName>body_link</bodyName>
+        <bodyName>base_link</bodyName>
         <topicName>fix</topicName>
         <velocityTopicName>fix_velocity</velocityTopicName>
@@ -55,5 +55,5 @@
         <alwaysOn>true</alwaysOn>
         <updateRate>100.0</updateRate>
-        <bodyName>body_link</bodyName>
+        <bodyName>base_link</bodyName>
         <topicName>ground_truth/state</topicName>
         <gaussianNoise>0.0</gaussianNoise>
@@ -63,5 +63,5 @@
 	<alwaysOn>true</alwaysOn>
 	<updateRate>10.0</updateRate>
-	<bodyName>body_link</bodyName>
+	<bodyName>base_link</bodyName>
 	<remoteModelName>robot</remoteModelName>
 	<remoteBodyName>base_link</remoteBodyName>

File: falkor_quadrotor_urdf/urdf/boy.urdf.xacro (robot description, xacro)
@@ -9,5 +9,5 @@
   <include filename="$(find falkor_quadrotor_urdf)/urdf/beacon_sensors.urdf.xacro" />
   <xacro:macro name="boy_base" params="mass height width depth">
-    <link name="body_link">
+    <link name="base_link">
       <inertial>
         <mass value="${mass}" />
