Commit message: centralize base sensors in its own urdf.xacro file

File: falkor_quadrotor_urdf/urdf/base_sensors.urdf.xacro (robot description, xacro)
@@ -5,6 +5,6 @@
 xmlns:xacro="http://ros.org/wiki/xacro"
 >
-  <!-- Quadrotor Sensor Plugins -->
-  <xacro:macro name="quadrotor_sensors">
+  <!-- Base Sensor Plugins -->
+  <xacro:macro name="base_sensors" params="tf_prefix">
     <gazebo>
       <controller:hector_gazebo_ros_imu name="quadrotor_imu_sim" plugin="libhector_gazebo_ros_imu.so">
@@ -15,10 +15,10 @@
         <rpyOffsets>0 0 0</rpyOffsets> <!-- deprecated -->
         <gaussianNoise>0</gaussianNoise>  <!-- deprecated -->
-        <accelDrift>0.5 0.5 0.5</accelDrift>
-        <accelGaussianNoise>0.35 0.35 0.3</accelGaussianNoise>
-        <rateDrift>0.1 0.1 0.1</rateDrift>
-        <rateGaussianNoise>0.05 0.05 0.015</rateGaussianNoise>
-        <headingDrift>0.1</headingDrift>
-        <headingGaussianNoise>0.05</headingGaussianNoise>
+        <accelDrift>0.1 0.1 0.1</accelDrift>
+        <accelGaussianNoise>0.05 0.05 0.05</accelGaussianNoise>
+        <rateDrift>0.02 0.02 0.02</rateDrift>
+        <rateGaussianNoise>0.005 0.005 0.005</rateGaussianNoise>
+        <headingDrift>0.01</headingDrift>
+        <headingGaussianNoise>0.01</headingGaussianNoise>
 	<frameId>/robot/imu</frameId>
       </controller:hector_gazebo_ros_imu>
@@ -30,6 +30,6 @@
         <altimeterTopicName>altimeter</altimeterTopicName>
         <offset>0</offset>
-        <drift>0.1</drift>
-        <gaussianNoise>0.5</gaussianNoise>
+        <drift>0.01</drift>
+        <gaussianNoise>0.05</gaussianNoise>
       </controller:hector_gazebo_ros_baro>
       <controller:hector_gazebo_ros_magnetic name="quadrotor_magnetic_sim" plugin="libhector_gazebo_ros_magnetic.so">
@@ -40,5 +40,5 @@
         <offset>0 0 0</offset>
         <drift>0.0 0.0 0.0</drift>
-        <gaussianNoise>1.3e-2 1.3e-2 1.3e-2</gaussianNoise>
+        <gaussianNoise>1.3e-3 1.3e-3 1.3e-3</gaussianNoise>
 	<!-- for zip code 11234
 	     from http://www.ngdc.noaa.gov/geomagmodels/struts/calcIGRFWMM
@@ -55,8 +55,8 @@
         <topicName>fix</topicName>
         <velocityTopicName>fix_velocity</velocityTopicName>
-        <drift>5.0 5.0 5.0</drift>
-        <gaussianNoise>0.1 0.1 0.1</gaussianNoise>
+        <drift>0.1 0.1 0.1</drift>
+        <gaussianNoise>0.01 0.01 0.01</gaussianNoise>
         <velocityDrift>0 0 0</velocityDrift>
-        <velocityGaussianNoise>0.1 0.1 0.1</velocityGaussianNoise>
+        <velocityGaussianNoise>0.01 0.01 0.01</velocityGaussianNoise>
 	<!-- RCSMP Marine Park, Brooklyn, NY -->
 	<referenceLatitude>40.589681</referenceLatitude>

File: falkor_quadrotor_urdf/urdf/beacon_sensors.urdf.xacro (robot description, xacro)
@@ -8,72 +8,4 @@
   <xacro:macro name="beacon_sensors">
     <gazebo>
-      <controller:hector_gazebo_ros_imu name="beacon_imu_sim" plugin="libhector_gazebo_ros_imu.so">
-        <alwaysOn>true</alwaysOn>
-        <updateRate>100.0</updateRate>
-        <bodyName>base_link</bodyName>
-        <topicName>raw_imu</topicName>
-        <rpyOffsets>0 0 0</rpyOffsets> <!-- deprecated -->
-        <gaussianNoise>0</gaussianNoise>  <!-- deprecated -->
-        <accelDrift>0.5 0.5 0.5</accelDrift>
-        <accelGaussianNoise>0.35 0.35 0.3</accelGaussianNoise>
-        <rateDrift>0.1 0.1 0.1</rateDrift>
-        <rateGaussianNoise>0.05 0.05 0.015</rateGaussianNoise>
-        <headingDrift>0.1</headingDrift>
-        <headingGaussianNoise>0.05</headingGaussianNoise>
-	<frameId>/beacon/imu</frameId>
-      </controller:hector_gazebo_ros_imu>
-      <controller:hector_gazebo_ros_baro name="beacon_baro_sim" plugin="libhector_gazebo_ros_baro.so">
-        <alwaysOn>true</alwaysOn>
-        <updateRate>10.0</updateRate>
-        <bodyName>base_link</bodyName>
-        <topicName>pressure_height</topicName>
-        <altimeterTopicName>altimeter</altimeterTopicName>
-        <offset>0</offset>
-        <drift>0.1</drift>
-        <gaussianNoise>0.5</gaussianNoise>
-      </controller:hector_gazebo_ros_baro>
-      <controller:hector_gazebo_ros_magnetic name="beacon_magnetic_sim" plugin="libhector_gazebo_ros_magnetic.so">
-        <alwaysOn>true</alwaysOn>
-        <updateRate>10.0</updateRate>
-        <bodyName>base_link</bodyName>
-        <topicName>magnetic</topicName>
-        <offset>0 0 0</offset>
-        <drift>0.0 0.0 0.0</drift>
-        <gaussianNoise>1.3e-2 1.3e-2 1.3e-2</gaussianNoise>
-	<!-- for zip code 11234
-	     from http://www.ngdc.noaa.gov/geomagmodels/struts/calcIGRFWMM
-	-->
-	<declination>-13.083</declination>
-	<inclination>66.867</inclination>
-	<!-- for zip code 11234
-	     from http://www.ngdc.noaa.gov/geomagmodels/struts/calcIGRFWMM
-	-->
-	<referenceHeading>0</referenceHeading>
-	<frameId>/beacon/magnetometer</frameId>
-      </controller:hector_gazebo_ros_magnetic>
-      <controller:hector_gazebo_ros_gps name="beacon_gps_sim" plugin="libhector_gazebo_ros_gps.so">
-        <alwaysOn>true</alwaysOn>
-        <updateRate>4.0</updateRate>
-        <bodyName>base_link</bodyName>
-        <topicName>fix</topicName>
-        <velocityTopicName>fix_velocity</velocityTopicName>
-        <drift>5.0 5.0 5.0</drift>
-        <gaussianNoise>0.1 0.1 0.1</gaussianNoise>
-        <velocityDrift>0 0 0</velocityDrift>
-        <velocityGaussianNoise>0.1 0.1 0.1</velocityGaussianNoise>
-	<!-- RCSMP Marine Park, Brooklyn, NY -->
-	<referenceLatitude>40.589681</referenceLatitude>
-	<referenceLongitude>-73.918520</referenceLongitude>
-	<referenceAltitude>0</referenceAltitude>
-	<referenceHeading>0</referenceHeading>
-      </controller:hector_gazebo_ros_gps>
-      <controller:gazebo_ros_p3d name="beacon_groundtruth_sim" plugin="libgazebo_ros_p3d.so">
-        <alwaysOn>true</alwaysOn>
-        <updateRate>100.0</updateRate>
-        <bodyName>base_link</bodyName>
-        <topicName>ground_truth/state</topicName>
-        <gaussianNoise>0.0</gaussianNoise>
-        <frameName>map</frameName>
-      </controller:gazebo_ros_p3d>
       <controller:falkor_quadrotor_sonar name="falkor_quadrotor_sonar" plugin="libfalkor_quadrotor_sonar.so">
 	<alwaysOn>true</alwaysOn>
@@ -82,5 +14,5 @@
 	<remoteModelName>robot</remoteModelName>
 	<remoteBodyName>base_link</remoteBodyName>
-	<gaussianNoise>0.05</gaussianNoise>
+	<gaussianNoise>0.01</gaussianNoise>
       </controller:falkor_quadrotor_sonar>
     </gazebo>

File: falkor_quadrotor_urdf/urdf/boy.urdf.xacro (robot description, xacro)
@@ -8,4 +8,5 @@
   <property name="pi" value="3.1415926535897931" />
   <include filename="$(find falkor_quadrotor_urdf)/urdf/beacon_sensors.urdf.xacro" />
+  <include filename="$(find falkor_quadrotor_urdf)/urdf/base_sensors.urdf.xacro" />
   <xacro:macro name="boy_base" params="mass height width depth">
     <link name="base_link">
@@ -39,4 +40,5 @@
     </gazebo>
     <beacon_sensors />
+    <base_sensors tf_prefix="/beacon" />
   </xacro:macro>
   <boy_base height="1.70" width="0.80" depth="0.60" mass="70" />

File: falkor_quadrotor_urdf/urdf/quadrotor_plugins.urdf.xacro (robot description, xacro)
@@ -1,10 +1,10 @@
 <?xml version="1.0"?>
 <robot xmlns:xacro="http://ros.org/wiki/xacro">
-  <xacro:include filename="$(find falkor_quadrotor_urdf)/urdf/quadrotor_sensors.urdf.xacro" />
+  <xacro:include filename="$(find falkor_quadrotor_urdf)/urdf/base_sensors.urdf.xacro" />
   <xacro:include filename="$(find falkor_quadrotor_urdf)/urdf/quadrotor_simple_controller.urdf.xacro" />
   <!-- Quadrotor Gazebo Plugins -->
   <xacro:macro name="quadrotor_plugins">
     <canonicalBody>base_link</canonicalBody>
-    <quadrotor_sensors/>
+    <base_sensors tf_prefix="/robot" />
     <quadrotor_controller/>
   </xacro:macro>
