Commit message: make combinegpsrawimu publish position->stabilized->link transform

File: falkor_quadrotor_urdf/urdf/quadrotor_base.urdf.xacro (robot description, xacro)
@@ -31,5 +31,5 @@
     <!-- Sonar height sensor -->
     <sonar_sensor name="sonar" parent="base_link" ros_topic="sonar_height" update_rate="10" min_range="0.03" max_range="3.0" field_of_view="40" ray_count="3" tf_prefix="/robot">
-      <origin xyz="0.12 0.0 -0.012" rpy="0 ${90*pi/180} 0"/>
+      <origin xyz="-0.25 0.0 0.20" rpy="0 ${90*pi/180} 0"/>
     </sonar_sensor>
     <gazebo reference="base_link">
