Commit message: some controller cleanups

File: falkor_quadrotor_urdf/urdf/generic_camera.urdf.xacro (robot description, xacro)
@@ -7,5 +7,5 @@
     <property name="M_PI" value="3.1415926535897931" />
     <xacro:macro name="generic_camera" params="name parent *origin ros_topic cam_info_topic update_rate res_x res_y image_format hfov tf_prefix">
-      <joint name="${name}_roll" type="continuous">
+      <joint name="${name}_roll" type="revolute">
         <insert_block name="origin" />
         <parent link="${parent}"/>
@@ -21,5 +21,5 @@
 	</inertial>
       </link>
-      <joint name="${name}_pitch" type="continuous">
+      <joint name="${name}_pitch" type="revolute">
         <insert_block name="origin" />
         <parent link="${name}_interm_link"/>

Commit message: fix a bunch of transforms

File: falkor_quadrotor_urdf/urdf/generic_camera.urdf.xacro (robot description, xacro)
@@ -22,5 +22,5 @@
       </link>
       <joint name="${name}_pitch" type="revolute">
-        <insert_block name="origin" />
+        <origin xyz="0 0 0" rpy="0 0 0" />
         <parent link="${name}_interm_link"/>
         <child link="${name}_link"/>

File: falkor_quadrotor_urdf/urdf/quadrotor_base.urdf.xacro (robot description, xacro)
@@ -31,5 +31,5 @@
     <!-- Sonar height sensor -->
     <sonar_sensor name="sonar" parent="base_link" ros_topic="sonar_height" update_rate="10" min_range="0.03" max_range="3.0" field_of_view="40" ray_count="3" tf_prefix="/robot">
-      <origin xyz="-0.25 0.0 0.20" rpy="0 ${90*pi/180} 0"/>
+      <origin xyz="0.0 0.0 0.20" rpy="0 ${90*pi/180} 0"/>
     </sonar_sensor>
     <gazebo reference="base_link">

File: falkor_quadrotor_urdf/urdf/quadrotor_with_cam.urdf.xacro (robot description, xacro)
@@ -18,5 +18,5 @@
     <include filename="$(find falkor_quadrotor_urdf)/urdf/generic_camera.urdf.xacro" />
     <xacro:generic_camera name="front_cam" parent="base_link" ros_topic="camera/image" cam_info_topic="camera/camera_info" update_rate="10" res_x="320" res_y="240" image_format="R8G8B8" hfov="90" tf_prefix="robot">
-      <origin xyz="0.05 0.0 -0.06" rpy="0 0 0"/>
+      <origin xyz="0.05 0.0 -0.15" rpy="0 0 0"/>
     </xacro:generic_camera>
 </robot>
